File: extension_board_10pin_molex_header/noname.kicad_pcb (KiCad board)
At the start: 2 copper layers, 18 x 39 mm, 4 parts, among them P1 CONN_02X05, P2 CONN_02X05

Commit message: Added 3d render
Parts:
- removed P2: CONN_02X05, Connectors_Molex:Connector_Microfit3_Header_02x05_Angled_43045-100x
- added P1: CONN_02X05, Connectors_Molex:Connector_Microfit3_Header_02x05_Angled_43045-100x, F.Cu at (115.0, 128.0)
Routing:
- net Net-(P1-Pad6): track 21.2 -> 20.3 mm
- net Net-(P1-Pad7): track 26.9 -> 26.0 mm
