File: main_master_board/_saved_main_master_board.sch (KiCad schematic (older format))
At the start: 1 part

Commit message: Added libraries for the Bucks we will be using
Connections:
- net labels added: +12V, +24V, +5V, VAA, VEE, VPP
- wire segments 53 -> 49
Changed lines of the file:
@@
 LIBS:USB_CONSOL-SchDoc-cache
 LIBS:VBAT_PROTECTION_REGS-SchDoc-cache
+LIBS:LMR16020
+LIBS:TPS832130SIL
 LIBS:main_master_board-cache
 EELAYER 25 0
@@
 $Descr A4 11693 8268
 encoding utf-8
-Sheet 1 1
+Sheet 1 2
 Title ""
 Date ""
@@
 NoConn ~ 18840 1860
 $Comp
-L VCC #PWR?
-U 1 1 58094BDB
-P 710 700
-F 0 "#PWR?" H 710 550 50  0001 C CNN
-F 1 "VCC" H 710 850 50  0000 C CNN
-F 2 "" H 710 700 50  0000 C CNN
-F 3 "" H 710 700 50  0000 C CNN
-	1    710  700
-	1    0    0    -1
-$EndComp
-$Comp
 L +3V3 #PWR?
 U 1 1 58094C11
-P 710 800
-F 0 "#PWR?" H 710 650 50  0001 C CNN
-F 1 "+3V3" H 710 940 50  0000 C CNN
-F 2 "" H 710 800 50  0000 C CNN
-F 3 "" H 710 800 50  0000 C CNN
-	1    710  800
-	-1   0    0    1
-$EndComp
-Wire Wire Line
-	18570 970  18570 1310
-Wire Wire Line
-	18570 1310 18570 1420
-Wire Wire Line
-	18570 1420 18570 1530
-Wire Wire Line
-	18550 5490 18550 5600
-Wire Wire Line
-	18550 5600 18550 5710
-Wire Wire Line
-	18550 5710 18550 5820
-Wire Wire Line
-	18550 5820 18550 5930
-Wire Wire Line
-	18550 5930 18550 6040
-Wire Wire Line
-	18550 6040 18550 6330
+P 1380 800
+F 0 "#PWR?" H 1380 650 50  0001 C CNN
+F 1 "+3V3" H 1380 940 50  0000 C CNN
+F 2 "" H 1380 800 50  0000 C CNN
+F 3 "" H 1380 800 50  0000 C CNN
+	1    1380 800
+	-1   0    0    1
+$EndComp
+Wire Wire Line
+	18570 970  18570 1530
+Wire Wire Line
+	18550 5490 18550 6330
 Wire Wire Line
 	18570 1310 18840 1310
@@
 $EndComp
 Wire Wire Line
-	710  700  710  800
+	1380 700  1380 800
 Wire Wire Line
 	920  700  920  790
@@
 L VDD #PWR?
 U 1 1 58224B23
-P 1140 700
-F 0 "#PWR?" H 1140 550 50  0001 C CNN
-F 1 "VDD" H 1140 850 50  0000 C CNN
-F 2 "" H 1140 700 50  0000 C CNN
-F 3 "" H 1140 700 50  0000 C CNN
-	1    1140 700
+P 1880 700
+F 0 "#PWR?" H 1880 550 50  0001 C CNN
+F 1 "VDD" H 1880 850 50  0000 C CNN
+F 2 "" H 1880 700 50  0000 C CNN
+F 3 "" H 1880 700 50  0000 C CNN
+	1    1880 700
 	1    0    0    -1
 $EndComp
@@
 Text Label 21450 6040 0    60   ~ 0
 I2C_1_SCL
+$Sheet
+S 2150 2450 820  710
+U 58643B62
+F0 "Power_conversion" 60
+F1 "Power_conversion.sch" 60
+F2 "V24_in" I L 2150 2670 60
+F3 "GND" I L 2150 2930 60
+F4 "V12_out" I R 2970 2550 60
+F5 "3V3_out" I R 2970 3030 60
+F6 "V5_out" I R 2970 2810 60
+$EndSheet
+$Comp
+L VCC #PWR?
+U 1 1 58643DBD
+P 660 710
+F 0 "#PWR?" H 660 560 50  0001 C CNN
+F 1 "VCC" H 660 860 50  0000 C CNN
+F 2 "" H 660 710 50  0000 C CNN
+F 3 "" H 660 710 50  0000 C CNN
+	1    660  710
+	1    0    0    -1
+$EndComp
+Wire Wire Line
+	660  710  660  810
+Wire Wire Line
+	1880 700  1880 800
+Wire Wire Line
+	1610 700  1610 800
+$Comp
+L +24V #PWR?
+U 1 1 58643E79
+P 660 810
+F 0 "#PWR?" H 660 660 50  0001 C CNN
+F 1 "+24V" H 660 950 50  0000 C CNN
+F 2 "" H 660 810 50  0000 C CNN
+F 3 "" H 660 810 50  0000 C CNN
+	1    660  810
+	-1   0    0    1
+$EndComp
+$Comp
+L +5V #PWR?
+U 1 1 586440F8
+P 1610 800
+F 0 "#PWR?" H 1610 650 50  0001 C CNN
+F 1 "+5V" H 1610 940 50  0000 C CNN
+F 2 "" H 1610 800 50  0000 C CNN
+F 3 "" H 1610 800 50  0000 C CNN
+	1    1610 800
+	-1   0    0    1
+$EndComp
+$Comp
+L +12V #PWR?
+U 1 1 5864412C
+P 1880 800
+F 0 "#PWR?" H 1880 650 50  0001 C CNN
+F 1 "+12V" H 1880 940 50  0000 C CNN
+F 2 "" H 1880 800 50  0000 C CNN
+F 3 "" H 1880 800 50  0000 C CNN
+	1    1880 800
+	-1   0    0    1
+$EndComp
+$Comp
+L VAA #PWR?
+U 1 1 58644259
+P 1380 700
+F 0 "#PWR?" H 1380 550 50  0001 C CNN
+F 1 "VAA" H 1380 850 50  0000 C CNN
+F 2 "" H 1380 700 50  0000 C CNN
+F 3 "" H 1380 700 50  0000 C CNN
+	1    1380 700
+	1    0    0    -1
+$EndComp
+$Comp
+L VEE #PWR?
+U 1 1 5864428D
+P 1610 700
+F 0 "#PWR?" H 1610 550 50  0001 C CNN
+F 1 "VEE" H 1610 850 50  0000 C CNN
+F 2 "" H 1610 700 50  0000 C CNN
+F 3 "" H 1610 700 50  0000 C CNN
+	1    1610 700
+	1    0    0    -1
+$EndComp
+$Comp
+L VPP #PWR?
+U 1 1 586442EC
+P 1140 700
+F 0 "#PWR?" H 1140 550 50  0001 C CNN
+F 1 "VPP" H 1140 850 50  0000 C CNN
+F 2 "" H 1140 700 50  0000 C CNN
+F 3 "" H 1140 700 50  0000 C CNN
+	1    1140 700
+	1    0    0    -1
+$EndComp
 $EndSCHEMATC
