File: main_master_board/Power_conversion.sch (KiCad schematic (older format))
At the start: 87 parts, among them IC1 IC_MCP73831, U10 FDS4935A, U11 Si1900DL, U12 FDS4935A, U2 LP3852-3.3, U3 TPS832130SIL, U4 LMR16020, U5 Si1900DL, U6 INA197, U7 INA197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

Commit message: Updating the footprints and components list. still working on it
Parts:
- C12: footprint (none) -> Capacitors_SMD:C_0603
- R1, R10, R16, R17, R2, R22, R25, R28, R31, R36, R5, R6, R8, R9: footprint (none) -> Resistors_SMD:R_0603
- R13, R18, R21, R3, R33: footprint Rled -> Resistors_SMD:R_0603
- R14, R23, R34: footprint Rreft -> Resistors_SMD:R_0603
- R15, R24, R35: footprint Rrefb -> Resistors_SMD:R_0603
- R7: footprint Rup -> Resistors_SMD:R_0603
- U6, U7, U8: symbol INA197 -> INA197-RESCUE-main_master_board
Connections:
- wire segments 382 -> 283

Commit message: I did a lot of things
Parts:
- C13, C15, C16: footprint Cin -> Capacitors_SMD:C_0805; Field5 (none) -> LMK212BJ106KG-T
- C17: footprint Cin2 -> Capacitors_SMD:C_0402; Field5 (none) -> GRM155R60J104KA01D
- C18: footprint Cvcc -> Capacitors_SMD:C_0603; Field4 (none) -> d; Field5 (none) -> GRM188R61A225KE34D
- C19: footprint (none) -> Capacitors_SMD:C_0603
- C20: footprint Ccomp2 -> Capacitors_SMD:C_0402; Field4 (none) -> d; Field5 (none) -> GRM1555C1H9R1CA01D
- C21: footprint Ccomp -> Capacitors_SMD:C_0201; Field4 (none) -> d; Field5 (none) -> GRM033R71C181KA01D
- C22: footprint Cbst -> Capacitors_SMD:C_0402; Field5 (none) -> GRM155R61A104KA01D
- C23, C24: footprint Cout -> Capacitors_SMD:C_1206; Field5 (none) -> GRM31CR71E106KA12L
- D10, D7, D8: footprint (none) -> SLP1006P2:SLP1006P2
- D11, D12: footprint VLMB1310-GS08CT-ND -> LEDs:LED_0603
- D4, D9: footprint 754-1126-1-ND -> LEDs:LED_0603
- D5: footprint 732-4978-1-ND -> LEDs:LED_0603
- F2: footprint (none) -> PTS181212V150:PTS181212
- F3, F4: footprint (none) -> SMD-1812:SMD-1812
- L2: footprint (none) -> IHLP-1616BZ:IHLP-1616BZ-11; Field5 (none) -> IHLP1616BZERR47M11
- R26: footprint Rcomp -> Resistors_SMD:R_0402; Field4 (none) -> d; Field5 (none) -> CRCW040269K8FKED
- R27: footprint Rlim -> Resistors_SMD:R_1206; Field4 (none) -> d; Field5 (none) -> ERJ-8ENF1583V
- R29: footprint Rfbt -> Resistors_SMD:R_0402; Field4 (none) -> d; Field5 (none) -> CRCW04021M05FKED
- R30: footprint Rfbb -> Resistors_SMD:R_0402; Field4 (none) -> d; Field5 (none) -> CRCW0402118KFKED
- R32: footprint Rt -> Resistors_SMD:R_1206; Field4 (none) -> d; Field5 (none) -> RC1206FR-0782KL
- S1: footprint (none) -> spdt:SPDT
- U10, U12: footprint (none) -> dp_devices:dp_devices-SO-8
- U11, U5: footprint MODULE -> NASA_IRG_SSB:SOT323-6
- U2: footprint MODULE -> SOT-223:SOT-223
- U6, U7, U8: footprint (none) -> dp_devices:dp_devices-SOT-23-5
- U9: footprint MODULE -> VQFN-11:VQFN-11

Commit message: Updated the project to no longer suppor the 12V Eragon board
Parts:
- removed C2: 10uF, Capacitors_SMD:C_1206, symbol C
- removed C3: 100nF, Capacitors_SMD:C_0603, symbol C_Small
- removed C5: 620pF, Capacitors_SMD:C_0402, symbol C
- removed C9: 22uF, Capacitors_SMD:C_0805, symbol C
- removed D5: RED_LED, LEDs:LED_0603, symbol LED-RESCUE-main_master_board
- removed D7: UCLAMP1211P, SLP1006P2:SLP1006P2, symbol D_TVS
- removed F2: PTS181212V150, PTS181212V150:PTS181212, symbol Fuse_Small
- removed R1: 10k, Resistors_SMD:R_0603, symbol R_Small
- removed R10: 100K, Resistors_SMD:R_0603, symbol R
- removed R11: 523K, Resistors_SMD:R_0402, symbol R
- removed R12: 100K, Resistors_SMD:R_0402, symbol R
- removed R13: 200, Resistors_SMD:R_0603, symbol R
- removed R14, R24: 102K, Resistors_SMD:R_0603, symbol R
- removed R15: 68.1K, Resistors_SMD:R_0603, symbol R
- removed R16: 0.02, Resistors_SMD:R_0603, symbol R
- removed R2: 2K, Resistors_SMD:R_0603, symbol R_Small
- removed R23: 267K, Resistors_SMD:R_0603, symbol R
- removed U3: TPS832130SIL, uSIP-8:uSIP-8, symbol TPS832130SIL
- removed U4: LMR16020, HSOIC-8:HSOIC-8-1EP_Pitch1.27mm, symbol LMR16020
- removed U6: INA197, dp_devices:dp_devices-SOT-23-5, symbol INA197-RESCUE-main_master_board
- added R?: 102K, Resistors_SMD:R_0603, symbol R
- added R?: 196K, Resistors_SMD:R_0603, symbol R
- added U4: LMR16030, HSOIC-8:HSOIC-8-1EP_Pitch1.27mm, symbol LMR16030
- C10: footprint Capacitors_SMD:C_0402 -> Capacitors_SMD:C_0805; Field5 C1005X7R1H104K -> C0805C104K5RACTU; Resistance 4.44mOhms -> 64mOhms
- C11: value 12pF -> 27pF; footprint Capacitors_SMD:C_0201 -> Capacitors_SMD:C_0805; Field5 C0201C120K3GACTU -> C0805C270J5GACTU; Resistance (none) -> 0.161Ohm; Voltage 25V -> (none)
- C14: value 4.7uF -> 33uF; Field5 GRM21BR61E475MA12L -> C2012X5R1A336M125AC; Resistance 2mOhms -> 1.69mOhms
- C4: footprint Capacitors_SMD:C_0603 -> Capacitors_SMD:C_0402; Field5 GRM31CR71H225KA88L -> C1005X5R1V225K050BC; Resistance 4.44mOhms -> 5.92mOhms
- L1: value 4.7uH -> 15uH; Field5 XAL4030-472MEB -> SRN8040-150M; Resistance 0.04 Ohm -> 0.07 Ohm
- R19: value 150K -> 68K; footprint Resistors_SMD:R_0402 -> Resistors_SMD:R_0603; Field5 CRCW0402150KFKED -> RC0603FR-0768KL
- R20: value 10K -> 12K; footprint Resistors_SMD:R_0402 -> Resistors_SMD:R_0603; Field5 CRCW040210K0FKED -> RC0603FR-0712KL
- R4: value 10.5K -> 45.3K; Field5 CRCW040210K5FKED -> CRCW040245K3FKED
Connections:
- net labels removed: V12, V12_FUSE, V12_cur, V12_out, V12_volt, v12_good, v5_ref
- wire segments 283 -> 228
Other:
- note removed: "12V to 5V Buck"
- moved on the sheet: C1, C8, D4, R3, U2

Commit message: Didn't save before pushing last commit
Parts:
- removed C13, C15, C16: 10uF, Capacitors_SMD:C_0805, symbol C_Small
- removed C17, C22: 100nF, Capacitors_SMD:C_0402, symbol C_Small
- removed C18: 2.2uF, Capacitors_SMD:C_0603, symbol C_Small
- removed C20: 9.10pF, Capacitors_SMD:C_0402, symbol C_Small
- removed C21: 180pF, Capacitors_SMD:C_0201, symbol C_Small
- removed C23, C24: 10uF, Capacitors_SMD:C_1206, symbol C_Small
- removed L2: 470nH, IHLP-1616BZ:IHLP-1616BZ-11, symbol L
- removed R26: 69.8K, Resistors_SMD:R_0402, symbol R
- removed R27: 158K, Resistors_SMD:R_1206, symbol R
- removed R29: 1.05M, Resistors_SMD:R_0402, symbol R
- removed R30: 118K, Resistors_SMD:R_0402, symbol R
- removed R32: 82K, Resistors_SMD:R_1206, symbol R
- removed U9: TPS61089, VQFN-11:VQFN-11, symbol TPS61089
- added C2: 22uF, Capacitors_SMD:C_0805, symbol C
- added C3: 15nF, Capacitors_SMD:C_0402, symbol C
- added C5: 47uF, Capacitors_SMD:C_1206, symbol C
- added L3: 1uH, IHLP-2020BZ:IHLP-2020BZ, symbol L
- added R10: 10K, Resistors_SMD:R_0603, symbol R_Small
- added U3: TPS61232DRC, Housings_DFN_QFN:DFN-10-1EP_3x3mm_Pitch0.5mm, symbol TPS61232DRC
- added U6: 74AUC1G32, SO-70:SO-70, symbol 74AUC1G32
- L1: footprint Inductors:Inductor_Wurth_MAPI-4020 -> Bourns:Bourns-8040
- gave numbers to parts that had none: 2
Connections:
- net labels added: PG_v5_backup, PG_v5_main, V5_BACKUP, V5_MAIN, V5_MERGE
- net labels removed: V12_BACKUP, V12_MAIN, V12_MERGE
- wire segments 228 -> 213
- no-connect marks 0 -> 1
Other:
- note removed: "4.2V to 12V Boost"
- note removed: "All the\nsame\ncapacitor"
- moved on the sheet: R34, R35
