File: main_master_board/snapdragon_edison.sch (KiCad schematic (older format))
At the start: 54 parts, among them J2 JD2-0011NL, U17 J1, U18 J2, U19 LAN9512, U21 MIC2026, U23 antenna, U24 AS1360, U25 Si1900DL, U26 SN74LV4T125, U27 SN74LV4T125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

Commit message: Started routing usb
Connections:
- net labels added: USBD2_N, USBD2_P, USBD3_N, USBD3_P
- net labels removed: USBDM2_N, USBDM3_N, USBDP2_P, USBDP3_P, USBPM3_N
Changed lines of the file:
@@
 PRTCTL3
 Text Label 7600 7350 0    60   ~ 0
-USBDP2_P
+USBD2_P
 Text Label 7600 7475 0    60   ~ 0
-USBDM2_N
+USBD2_N
 Text Label 7600 7650 0    60   ~ 0
-USBDP3_P
+USBD3_P
 Text Label 7600 7775 0    60   ~ 0
-USBPM3_N
+USBD3_N
 $Comp
 L R R30
@@
 Wire Wire Line
 	1600 3000 2050 3000
-Text Label 14675 4050 2    60   ~ 0
-USBDP2_P
-Text Label 14675 4150 2    60   ~ 0
-USBDM2_N
-Text Label 14675 4425 2    60   ~ 0
-USBDP3_P
-Text Label 14675 4525 2    60   ~ 0
-USBDM3_N
 Text Label 14675 2875 2    60   ~ 0
 I2C1_SCL
@@
 Text Label 10675 8650 0    60   ~ 0
 TX_N
+Text Label 14675 4050 2    60   ~ 0
+USBD2_P
+Text Label 14675 4150 2    60   ~ 0
+USBD2_N
+Text Label 14675 4425 2    60   ~ 0
+USBD3_P
+Text Label 14675 4525 2    60   ~ 0
+USBD3_N
 $EndSCHEMATC
