File: main_master_board/Power_Saftey_Switches.sch (KiCad schematic (older format))
At the start: 26 parts, among them P10 watchdog, P11 CONN_01X05, P12 motors_en, P9 uC_KS, Q1 PSMN013-80YS, Q2 LT1910, U13 74HC1G126, U14 PIC12(L)F1571/2

Commit message: Changed expansion connector to two connectors. Routed 5 to 4 buck.
Parts:
- P11: footprint SMD_pinheader:01x05_pinheader_SMD -> Pin_Headers:Pin_Header_Angled_1x05_Pitch1.27mm
- R42: footprint Resistors_SMD:R_0603 -> Resistors_SMD:R_1210
Changed lines of the file:
@@
 F 0 "R42" V 6780 1590 50  0000 C CNN
 F 1 "0.0025" V 6600 1590 50  0000 C CNN
-F 2 "Resistors_SMD:R_0603" V 6630 1590 50  0001 C CNN
+F 2 "Resistors_SMD:R_1210" V 6630 1590 50  0001 C CNN
 F 3 "" H 6700 1590 50  0000 C CNN
 	1    6700 1590
@@
 F 0 "P11" H 3930 5920 50  0000 C CNN
 F 1 "CONN_01X05" V 4030 5620 50  0000 C CNN
-F 2 "SMD_pinheader:01x05_pinheader_SMD" H 3930 5620 50  0001 C CNN
+F 2 "Pin_Headers:Pin_Header_Angled_1x05_Pitch1.27mm" H 3930 5620 50  0001 C CNN
 F 3 "" H 3930 5620 50  0000 C CNN
 F 4 "http://www.digikey.com/product-detail/en/3m/961105-6300-AR-PR/3M9487CT-ND/2071622" H 3930 5620 60  0001 C CNN "Field4"
