File: connectors.sch (KiCad schematic (older format))
At the start: 4 parts, among them P1 Vbackup, P2 CONN_02X05, P3 Hebi_1, P4 Hebi_2

Commit message: Moved library files to dedicated folder. Added support for Edison and Open-Q 410 boards.
Parts:
- added D2, D3: D_Schottky, TO-220-3:D-Pack-3, symbol D_Schottky
Connections:
- net labels added: Vmotors
- wire segments 22 -> 30
Other:
- note added: "Bettery Reverse\nCurrent Protection"
Changed lines of the file:
@@
 LIBS:USB_CONSOL-SchDoc-cache
 LIBS:VBAT_PROTECTION_REGS-SchDoc-cache
-LIBS:LMR16020
-LIBS:TPS832130SIL
 LIBS:TPS754
-LIBS:TPS61089
 LIBS:FDS4935A
 LIBS:Si1900DL
@@
 LIBS:xal6030-182mec
 LIBS:decaWave
+LIBS:conn_2x50
+LIBS:conn_open_q_x2
+LIBS:LMR16020
+LIBS:TPS61089
 LIBS:TPS61232DRC
+LIBS:TPS832130SIL
+LIBS:SS4-50-3.00-X-D
 LIBS:main_master_board-cache
 EELAYER 25 0
@@
 $Descr A4 11693 8268
 encoding utf-8
-Sheet 5 5
+Sheet 5 6
 Title ""
 Date ""
@@
 	1    0    0    -1
 $EndComp
-Text Label 2030 2320 2    60   ~ 0
+Text Label 2590 2320 0    60   ~ 0
 V24_in
-Text Label 2590 2720 0    60   ~ 0
+Text Label 2020 2720 2    60   ~ 0
 V24_in
-$Comp
-L GNDPWR #PWR015
-U 1 1 5876C3CF
-P 1980 2790
-F 0 "#PWR015" H 1980 2590 50  0001 C CNN
-F 1 "GNDPWR" H 1980 2660 50  0000 C CNN
-F 2 "" H 1980 2740 50  0000 C CNN
-F 3 "" H 1980 2740 50  0000 C CNN
-	1    1980 2790
-	1    0    0    -1
-$EndComp
 $Comp
 L GNDPWR #PWR016
 U 1 1 5876C3D5
-P 2760 2140
-F 0 "#PWR016" H 2760 1940 50  0001 C CNN
-F 1 "GNDPWR" H 2760 2010 50  0000 C CNN
-F 2 "" H 2760 2090 50  0000 C CNN
-F 3 "" H 2760 2090 50  0000 C CNN
-	1    2760 2140
-	1    0    0    -1
-$EndComp
-Wire Wire Line
-	2060 2320 1720 2320
-Wire Wire Line
-	2560 2720 2890 2720
-Wire Wire Line
-	2560 2320 2590 2320
-Wire Wire Line
-	2590 2320 2590 2140
-Wire Wire Line
-	2590 2140 2760 2140
-Wire Wire Line
-	2060 2720 1980 2720
-Wire Wire Line
-	1980 2720 1980 2790
+P 1840 2170
+F 0 "#PWR016" H 1840 1970 50  0001 C CNN
+F 1 "GNDPWR" H 1840 2040 50  0000 C CNN
+F 2 "" H 1840 2120 50  0000 C CNN
+F 3 "" H 1840 2120 50  0000 C CNN
+	1    1840 2170
+	1    0    0    -1
+$EndComp
 Wire Wire Line
 	2060 2420 1630 2420
@@
 Wire Wire Line
 	3950 3740 4330 3740
+Text HLabel 10340 1150 2    60   Output ~ 0
+V24_in
+Text HLabel 10340 1440 2    60   Output ~ 0
+Vbackup_in
+$Comp
+L D_Schottky D3
+U 1 1 587AC4FF
+P 3960 4550
+F 0 "D3" H 3960 4650 50  0000 C CNN
+F 1 "D_Schottky" H 3960 4450 50  0000 C CNN
+F 2 "TO-220-3:D-Pack-3" H 3960 4550 50  0001 C CNN
+F 3 "http://datasheet.octopart.com/STPS5H100B-TR-STMicroelectronics-datasheet-5318140.pdf" H 3960 4550 50  0001 C CNN
+	1    3960 4550
+	-1   0    0    1
+$EndComp
+Text Label 4150 4550 0    60   ~ 0
+V_hebi1
+$Comp
+L D_Schottky D2
+U 1 1 587AC507
+P 3950 4840
+F 0 "D2" H 3950 4940 50  0000 C CNN
+F 1 "D_Schottky" H 3950 4740 50  0000 C CNN
+F 2 "TO-220-3:D-Pack-3" H 3950 4840 50  0001 C CNN
+F 3 "http://datasheet.octopart.com/STPS5H100B-TR-STMicroelectronics-datasheet-5318140.pdf" H 3950 4840 50  0001 C CNN
+	1    3950 4840
+	-1   0    0    1
+$EndComp
+Text Label 4140 4840 0    60   ~ 0
+V_hebi2
+Text Notes 3520 4380 0    60   ~ 0
+Bettery Reverse\nCurrent Protection
+Text Label 3530 4550 0    60   ~ 0
+Vmotors
+Text Label 3520 4840 0    60   ~ 0
+Vmotors
+Wire Wire Line
+	3810 4550 3490 4550
+Wire Wire Line
+	4110 4550 4460 4550
+Wire Wire Line
+	3800 4840 3480 4840
+Wire Wire Line
+	4100 4840 4450 4840
+$Comp
+L GNDPWR #PWR020
+U 1 1 5876C3CF
+P 2680 2770
+F 0 "#PWR020" H 2680 2570 50  0001 C CNN
+F 1 "GNDPWR" H 2680 2640 50  0000 C CNN
+F 2 "" H 2680 2720 50  0000 C CNN
+F 3 "" H 2680 2720 50  0000 C CNN
+	1    2680 2770
+	1    0    0    -1
+$EndComp
+Wire Wire Line
+	2560 2720 2680 2720
+Wire Wire Line
+	2680 2720 2680 2770
+Wire Wire Line
+	2060 2720 1730 2720
+Wire Wire Line
+	2060 2320 2020 2320
+Wire Wire Line
+	2020 2320 2020 2140
+Wire Wire Line
+	2020 2140 1840 2140
+Wire Wire Line
+	1840 2140 1840 2170
+Wire Wire Line
+	2560 2320 2890 2320
+Wire Wire Line
+	10340 1150 10000 1150
+Wire Wire Line
+	10340 1440 9800 1440
+Text Label 10300 1440 2    60   ~ 0
+Vbackup_in
+Text Label 10300 1150 2    60   ~ 0
+V24_in
+Text HLabel 1030 800  0    60   Input ~ 0
+Vmotors
+Wire Wire Line
+	1030 800  1430 800
+Text Label 1050 800  0    60   ~ 0
+Vmotors
 $EndSCHEMATC

Commit message: Working on moving things to two boards
Parts:
- added D?: P6SMB30AT3G, Diodes_SMD:SMB_Standard, symbol ZENERsmall
- added F?: 3413.0328.22, dp_devices:dp_devices-C1206, symbol Fuse
- added J?: RJ45, symbol RJ45
- added P? (x2): CONN_01X04, microclasp_4:microclasp_4, symbol CONN_01X04
- added S?: SWITCH_DPDT, microclasp:microclasp_3, symbol SWITCH_DPDT
- added SW?: SWITCH_SPST, molex_microclasp2:microclasp_vdrx2, symbol SWITCH_SPST
Connections:
- net labels added: 3V3, KS_physical_in, KS_physical_out, KS_pysical_in, KS_pysical_out, Switch_on, V4, Vmain, uC_SCL, uC_SDA
- wire segments 30 -> 56
Other:
- note added: "AMS5600 Magnetic Rotary \nSensor Support\n"
- note added: "Circuits can take 48V, \nexcept TSV diode"
- note added: "Manual switch to \nturn motors off"
- note added: "TCS3472 Color Sensor Support\n"
- note added: "Transient Voltage Suppessor"
Changed lines of the file:
@@
 LIBS:FDS4935A
 LIBS:Si1900DL
-LIBS:Amplifiers
-LIBS:Connectors
-LIBS:DataStorage
-LIBS:Diodes
-LIBS:Microprocessors
-LIBS:MiscellaneousDevices
-LIBS:Passives
-LIBS:PMOD
-LIBS:PowerComponents
-LIBS:RepeaterParts
-LIBS:RF_OEM_Parts
 LIBS:Sensors
-LIBS:TransistorParts
 LIBS:LP3852-3.3
 LIBS:0s102011ma1qn1
@@
 LIBS:xal5050-562meb
 LIBS:xal6030-182mec
-LIBS:decaWave
 LIBS:conn_2x50
 LIBS:conn_open_q_x2
@@
 LIBS:ac-dc
 LIBS:actel
-LIBS:allegro
 LIBS:Altera
 LIBS:analog_devices
@@
 LIBS:logo
 LIBS:maxim
-LIBS:mechanical
 LIBS:microchip_dspic33dsc
 LIBS:microchip_pic10mcu
@@
 LIBS:microchip_pic32mcu
 LIBS:motor_drivers
-LIBS:motors
 LIBS:msp430
 LIBS:nordicsemi
@@
 LIBS:ttl_ieee
 LIBS:video
-LIBS:wiznet
 LIBS:Worldsemi
 LIBS:Xicor
-LIBS:zetex
 LIBS:Zilog
 LIBS:conn_2x45
@@
 	1    0    0    -1
 $EndComp
-Wire Wire Line
-	2060 2420 1630 2420
 Text Label 1640 2420 0    60   ~ 0
 signal_1s
-Wire Wire Line
-	2060 2520 1630 2520
-Wire Wire Line
-	2060 2620 1630 2620
 Text Label 1650 2520 0    60   ~ 0
 signal_3s
@@
 Text Label 2570 2420 0    60   ~ 0
 signal_2s
-Wire Wire Line
-	2560 2420 2990 2420
-Wire Wire Line
-	2560 2520 2990 2520
-Wire Wire Line
-	2560 2620 2990 2620
 Text Label 2570 2520 0    60   ~ 0
 signal_4s
@@
 	-1   0    0    1
 $EndComp
-Wire Wire Line
-	2080 3290 2590 3290
 Text Label 2090 3290 0    60   ~ 0
 Vbackup_in
@@
 	1    0    0    -1
 $EndComp
-Wire Wire Line
-	2080 3390 2130 3390
-Wire Wire Line
-	2130 3390 2130 3410
 $Comp
 L CONN_01X02 P3
@@
 	-1   0    0    1
 $EndComp
-Wire Wire Line
-	3950 3300 4320 3300
 Text Label 3970 3300 0    60   ~ 0
 V_hebi1
@@
 	1    0    0    -1
 $EndComp
-Wire Wire Line
-	3950 3840 4000 3840
-Wire Wire Line
-	4000 3840 4000 3870
-Wire Wire Line
-	3950 3400 4010 3400
-Wire Wire Line
-	4010 3400 4010 3430
 Text Label 3980 3740 0    60   ~ 0
 V_hebi2
-Wire Wire Line
-	3950 3740 4330 3740
 Text HLabel 10340 1150 2    60   Output ~ 0
 V24_in
@@
 Text Label 3520 4840 0    60   ~ 0
 Vmotors
-Wire Wire Line
-	3810 4550 3490 4550
-Wire Wire Line
-	4110 4550 4460 4550
-Wire Wire Line
-	3800 4840 3480 4840
-Wire Wire Line
-	4100 4840 4450 4840
 $Comp
 L GNDPWR #PWR021
@@
 	1    0    0    -1
 $EndComp
-Wire Wire Line
-	2560 2720 2680 2720
-Wire Wire Line
-	2680 2720 2680 2770
-Wire Wire Line
-	2060 2720 1730 2720
-Wire Wire Line
-	2060 2320 2020 2320
-Wire Wire Line
-	2020 2320 2020 2140
-Wire Wire Line
-	2020 2140 1840 2140
-Wire Wire Line
-	1840 2140 1840 2170
-Wire Wire Line
-	2560 2320 2890 2320
-Wire Wire Line
-	10340 1150 10000 1150
-Wire Wire Line
-	10340 1440 9800 1440
 Text Label 10300 1440 2    60   ~ 0
 Vbackup_in
@@
 Text HLabel 1030 800  0    60   Input ~ 0
 Vmotors
-Wire Wire Line
-	1030 800  1430 800
 Text Label 1050 800  0    60   ~ 0
 Vmotors
+$Comp
+L CONN_01X04 P?
+U 1 1 58811D9C
+P 7275 1325
+F 0 "P?" H 7275 1575 50  0000 C CNN
+F 1 "CONN_01X04" V 7375 1325 50  0000 C CNN
+F 2 "microclasp_4:microclasp_4" H 7275 1325 50  0001 C CNN
+F 3 "" H 7275 1325 50  0000 C CNN
+	1    7275 1325
+	1    0    0    -1
+$EndComp
+Text Label 7050 1175 2    60   ~ 0
+GND
+Text Label 7050 1275 2    60   ~ 0
+3V3
+Text Label 7050 1375 2    60   ~ 0
+uC_SCL
+Text Label 7050 1475 2    60   ~ 0
+uC_SDA
+Text Notes 6350 875  0    60   ~ 0
+AMS5600 Magnetic Rotary \nSensor Support\n
+$Comp
+L CONN_01X04 P?
+U 1 1 58811DAC
+P 7250 2025
+F 0 "P?" H 7250 2275 50  0000 C CNN
+F 1 "CONN_01X04" V 7350 2025 50  0000 C CNN
+F 2 "microclasp_4:microclasp_4" H 7250 2025 50  0001 C CNN
+F 3 "" H 7250 2025 50  0000 C CNN
+	1    7250 2025
+	1    0    0    -1
+$EndComp
+Text Label 7025 1875 2    60   ~ 0
+GND
+Text Label 7025 1975 2    60   ~ 0
+3V3
+Text Label 7025 2075 2    60   ~ 0
+uC_SCL
+Text Label 7025 2175 2    60   ~ 0
+uC_SDA
+Text Notes 6225 1700 0    60   ~ 0
+TCS3472 Color Sensor Support\n
+Text HLabel 1000 975  0    60   Input ~ 0
+3V3
+Text HLabel 1025 1375 0    60   Input ~ 0
+GND
+Text HLabel 1000 1575 0    60   Input ~ 0
+uC_SDA
+Text HLabel 1000 1725 0    60   Input ~ 0
+uC_SCL
+Text Label 1050 975  0    60   ~ 0
+3V3
+Text Label 1075 1375 0    60   ~ 0
+GND
+Text Label 1050 1575 0    60   ~ 0
+uC_SDA
+Text Label 1050 1725 0    60   ~ 0
+uC_SCL
+Wire Wire Line
+	2060 2420 1630 2420
+Wire Wire Line
+	2060 2520 1630 2520
+Wire Wire Line
+	2060 2620 1630 2620
+Wire Wire Line
+	2560 2420 2990 2420
+Wire Wire Line
+	2560 2520 2990 2520
+Wire Wire Line
+	2560 2620 2990 2620
+Wire Wire Line
+	2080 3290 2590 3290
+Wire Wire Line
+	2080 3390 2130 3390
+Wire Wire Line
+	2130 3390 2130 3410
+Wire Wire Line
+	3950 3300 4320 3300
+Wire Wire Line
+	3950 3840 4000 3840
+Wire Wire Line
+	4000 3840 4000 3870
+Wire Wire Line
+	3950 3400 4010 3400
+Wire Wire Line
+	4010 3400 4010 3430
+Wire Wire Line
+	3950 3740 4330 3740
+Wire Wire Line
+	3810 4550 3490 4550
+Wire Wire Line
+	4110 4550 4460 4550
+Wire Wire Line
+	3800 4840 3480 4840
+Wire Wire Line
+	4100 4840 4450 4840
+Wire Wire Line
+	2560 2720 2680 2720
+Wire Wire Line
+	2680 2720 2680 2770
+Wire Wire Line
+	2060 2720 1730 2720
+Wire Wire Line
+	2060 2320 2020 2320
+Wire Wire Line
+	2020 2320 2020 2140
+Wire Wire Line
+	2020 2140 1840 2140
+Wire Wire Line
+	1840 2140 1840 2170
+Wire Wire Line
+	2560 2320 2890 2320
+Wire Wire Line
+	10340 1150 10000 1150
+Wire Wire Line
+	10340 1440 9800 1440
+Wire Wire Line
+	1030 800  1430 800
+Wire Wire Line
+	7075 1175 6850 1175
+Wire Wire Line
+	7075 1275 6875 1275
+Wire Wire Line
+	6500 1375 7075 1375
+Wire Wire Line
+	6325 1475 7075 1475
+Wire Wire Line
+	7050 1875 6825 1875
+Wire Wire Line
+	7050 1975 6850 1975
+Wire Wire Line
+	7050 2075 6700 2075
+Wire Wire Line
+	7050 2175 6700 2175
+Wire Wire Line
+	1000 975  1225 975
+Wire Wire Line
+	1025 1375 1275 1375
+Wire Wire Line
+	1000 1575 1400 1575
+$Comp
+L SWITCH_SPST SW?
+U 1 1 58817B83
+P 6875 2900
+F 0 "SW?" H 6875 3050 60  0000 C CNN
+F 1 "SWITCH_SPST" V 6875 2580 60  0000 C CNN
+F 2 "molex_microclasp2:microclasp_vdrx2" H 6875 2900 60  0001 C CNN
+F 3 "" H 6875 2900 60  0000 C CNN
+	1    6875 2900
+	0    -1   -1   0
+$EndComp
+Wire Wire Line
+	6875 2700 7575 2700
+Text Label 6905 3100 0    60   ~ 0
+KS_physical_out
+Text Label 6905 2700 0    60   ~ 0
+KS_physical_in
+Text Notes 6865 2580 0    60   ~ 0
+Manual switch to \nturn motors off
+Wire Wire Line
+	6875 3100 7650 3100
+Wire Wire Line
+	1000 1725 1400 1725
+Text HLabel 1200 1900 0    60   Input ~ 0
+KS_pysical_in
+Wire Wire Line
+	1200 1900 1875 1900
+Text Label 1225 1900 0    60   ~ 0
+KS_physical_in
+Text HLabel 10350 1650 2    60   Output ~ 0
+KS_pysical_out
+Text Label 10325 1650 2    60   ~ 0
+KS_physical_out
+Wire Wire Line
+	10350 1650 9600 1650
+$Comp
+L SWITCH_DPDT S?
+U 1 1 5881AA8A
+P 5425 1300
+F 0 "S?" V 5305 950 60  0000 C CNN
+F 1 "SWITCH_DPDT" V 5305 1400 60  0000 C CNN
+F 2 "microclasp:microclasp_3" H 5425 1300 60  0001 C CNN
+F 3 "" H 5425 1300 60  0000 C CNN
+	1    5425 1300
+	0    1    1    0
+$EndComp
+Text Label 5105 1300 2    60   ~ 0
+V4
+Text Label 5745 1300 0    60   ~ 0
+GND
+Wire Wire Line
+	5125 1300 4925 1300
+Wire Wire Line
+	5725 1300 5945 1300
+Wire Wire Line
+	5425 1400 5425 1575
+Wire Wire Line
+	5425 1575 5950 1575
+Text Label 5475 1575 0    60   ~ 0
+Switch_on
+Text HLabel 1000 1125 0    60   Input ~ 0
+V4
+Text Label 1050 1125 0    60   ~ 0
+V4
+Wire Wire Line
+	1000 1125 1225 1125
+Text HLabel 10350 1850 2    60   Output ~ 0
+Switch_on
+Wire Wire Line
+	10350 1850 9875 1850
+Text Label 10325 1850 2    60   ~ 0
+Switch_on
+$Comp
+L RJ45 J?
+U 1 1 5881C2C5
+P 1925 4750
+F 0 "J?" H 2125 5250 50  0000 C CNN
+F 1 "RJ45" H 1775 5250 50  0000 C CNN
+F 2 "" H 1925 4750 50  0000 C CNN
+F 3 "" H 1925 4750 50  0000 C CNN
+	1    1925 4750
+	1    0    0    -1
+$EndComp
+$Comp
+L ZENERsmall D?
+U 1 1 58821700
+P 3220 1060
+F 0 "D?" H 3320 1020 50  0000 C CNN
+F 1 "P6SMB30AT3G" H 3360 1180 50  0000 C CNN
+F 2 "Diodes_SMD:SMB_Standard" H 3220 1060 50  0001 C CNN
+F 3 "http://datasheet.octopart.com/P6SMB36AT3G-ON-Semiconductor-datasheet-5314825.pdf" H 3220 1060 50  0001 C CNN
+	1    3220 1060
+	0    1    1    0
+$EndComp
+$Comp
+L GND #PWR?
+U 1 1 58821707
+P 3220 1220
+F 0 "#PWR?" H 3220 970 50  0001 C CNN
+F 1 "GND" H 3220 1070 50  0000 C CNN
+F 2 "" H 3220 1220 50  0000 C CNN
+F 3 "" H 3220 1220 50  0000 C CNN
+	1    3220 1220
+	1    0    0    -1
+$EndComp
+Text Notes 2580 1540 0    60   ~ 0
+Transient Voltage Suppessor
+Text Label 3300 920  0    60   ~ 0
+Vmain
+Text Notes 3410 1420 0    60   ~ 0
+Circuits can take 48V, \nexcept TSV diode
+Text Label 2520 920  0    60   ~ 0
+V24_in
+$Comp
+L Fuse F?
+U 1 1 58821711
+P 2950 920
+F 0 "F?" V 3030 920 50  0000 C CNN
+F 1 "3413.0328.22" V 2875 920 50  0000 C CNN
+F 2 "dp_devices:dp_devices-C1206" V 2880 920 50  0001 C CNN
+F 3 "http://datasheet.octopart.com/3413.0328.22-Schurter-datasheet-8645987.pdf" H 2950 920 50  0001 C CNN
+	1    2950 920
+	0    -1   -1   0
+$EndComp
+Wire Wire Line
+	3100 920  3740 920
+Wire Wire Line
+	3220 920  3220 960
+Connection ~ 3220 920
+Wire Wire Line
+	3220 1160 3220 1220
+Wire Wire Line
+	2800 920  2510 920
 $EndSCHEMATC

Commit message: Started working on design and layout for fulll board with dart410. Added Macrofab libraries
Parts:
- removed P? (x2): CONN_01X04, microclasp_4:microclasp_4, symbol CONN_01X04
- J1: renamed from J?; footprint (none) -> RJ45-SMD:TE-338088
- P1: footprint Battery_Holders:Keystone_2466_1xAAA -> microclasp:microclasp_2
- gave numbers to parts that had none: 4
Connections:
- wire segments 56 -> 48
Other:
- note removed: "AMS5600 Magnetic Rotary \nSensor Support\n"
- note removed: "TCS3472 Color Sensor Support\n"
Changed lines of the file:
@@
 LIBS:Zilog
 LIBS:conn_2x45
+LIBS:MF_Aesthetics
+LIBS:MF_Connectors
+LIBS:MF_Discrete_Semiconductor
+LIBS:MF_Displays
+LIBS:MF_Frequency_Control
+LIBS:MF_IC_Analog
+LIBS:MF_IC_Digital
+LIBS:MF_IC_Power
+LIBS:MF_LEDs
+LIBS:MF_Passives
+LIBS:MF_Sensors
+LIBS:MF_Switches
 LIBS:main_master_board-cache
 EELAYER 25 0
@@
 V24_in
 $Comp
-L GNDPWR #PWR017
+L GNDPWR #PWR016
 U 1 1 5876C3D5
 P 1840 2170
-F 0 "#PWR017" H 1840 1970 50  0001 C CNN
+F 0 "#PWR016" H 1840 1970 50  0001 C CNN
 F 1 "GNDPWR" H 1840 2040 50  0000 C CNN
 F 2 "" H 1840 2120 50  0000 C CNN
@@
 F 0 "P1" H 1880 3490 50  0000 C CNN
 F 1 "Vbackup" V 1980 3340 50  0000 C CNN
-F 2 "Battery_Holders:Keystone_2466_1xAAA" H 1880 3340 50  0001 C CNN
+F 2 "microclasp:microclasp_2" H 1880 3340 50  0001 C CNN
 F 3 "" H 1880 3340 50  0000 C CNN
 	1    1880 3340
@@
 Vbackup_in
 $Comp
-L GND #PWR018
+L GND #PWR017
 U 1 1 5876C3F8
 P 2130 3410
-F 0 "#PWR018" H 2130 3160 50  0001 C CNN
+F 0 "#PWR017" H 2130 3160 50  0001 C CNN
 F 1 "GND" H 2130 3260 50  0000 C CNN
 F 2 "" H 2130 3410 50  0000 C CNN
@@
 V_hebi1
 $Comp
-L GNDPWR #PWR019
+L GNDPWR #PWR018
 U 1 1 5876E2BA
 P 4010 3430
-F 0 "#PWR019" H 4010 3230 50  0001 C CNN
+F 0 "#PWR018" H 4010 3230 50  0001 C CNN
 F 1 "GNDPWR" H 4010 3300 50  0000 C CNN
 F 2 "" H 4010 3380 50  0000 C CNN
@@
 $EndComp
 $Comp
-L GNDPWR #PWR020
+L GNDPWR #PWR019
 U 1 1 5876E2C0
 P 4000 3870
-F 0 "#PWR020" H 4000 3670 50  0001 C CNN
+F 0 "#PWR019" H 4000 3670 50  0001 C CNN
 F 1 "GNDPWR" H 4000 3740 50  0000 C CNN
 F 2 "" H 4000 3820 50  0000 C CNN
@@
 Vmotors
 $Comp
-L GNDPWR #PWR021
+L GNDPWR #PWR020
 U 1 1 5876C3CF
 P 2680 2770
-F 0 "#PWR021" H 2680 2570 50  0001 C CNN
+F 0 "#PWR020" H 2680 2570 50  0001 C CNN
 F 1 "GNDPWR" H 2680 2640 50  0000 C CNN
 F 2 "" H 2680 2720 50  0000 C CNN
@@
 Text Label 1050 800  0    60   ~ 0
 Vmotors
-$Comp
-L CONN_01X04 P?
-U 1 1 58811D9C
-P 7275 1325
-F 0 "P?" H 7275 1575 50  0000 C CNN
-F 1 "CONN_01X04" V 7375 1325 50  0000 C CNN
-F 2 "microclasp_4:microclasp_4" H 7275 1325 50  0001 C CNN
-F 3 "" H 7275 1325 50  0000 C CNN
-	1    7275 1325
-	1    0    0    -1
-$EndComp
-Text Label 7050 1175 2    60   ~ 0
-GND
-Text Label 7050 1275 2    60   ~ 0
-3V3
-Text Label 7050 1375 2    60   ~ 0
-uC_SCL
-Text Label 7050 1475 2    60   ~ 0
-uC_SDA
-Text Notes 6350 875  0    60   ~ 0
-AMS5600 Magnetic Rotary \nSensor Support\n
-$Comp
-L CONN_01X04 P?
-U 1 1 58811DAC
-P 7250 2025
-F 0 "P?" H 7250 2275 50  0000 C CNN
-F 1 "CONN_01X04" V 7350 2025 50  0000 C CNN
-F 2 "microclasp_4:microclasp_4" H 7250 2025 50  0001 C CNN
-F 3 "" H 7250 2025 50  0000 C CNN
-	1    7250 2025
-	1    0    0    -1
-$EndComp
-Text Label 7025 1875 2    60   ~ 0
-GND
-Text Label 7025 1975 2    60   ~ 0
-3V3
-Text Label 7025 2075 2    60   ~ 0
-uC_SCL
-Text Label 7025 2175 2    60   ~ 0
-uC_SDA
-Text Notes 6225 1700 0    60   ~ 0
-TCS3472 Color Sensor Support\n
 Text HLabel 1000 975  0    60   Input ~ 0
 3V3
@@
 	1030 800  1430 800
 Wire Wire Line
-	7075 1175 6850 1175
-Wire Wire Line
-	7075 1275 6875 1275
-Wire Wire Line
-	6500 1375 7075 1375
-Wire Wire Line
-	6325 1475 7075 1475
-Wire Wire Line
-	7050 1875 6825 1875
-Wire Wire Line
-	7050 1975 6850 1975
-Wire Wire Line
-	7050 2075 6700 2075
-Wire Wire Line
-	7050 2175 6700 2175
-Wire Wire Line
 	1000 975  1225 975
 Wire Wire Line
@@
 	1000 1575 1400 1575
 $Comp
-L SWITCH_SPST SW?
+L SWITCH_SPST SW1
 U 1 1 58817B83
 P 6875 2900
-F 0 "SW?" H 6875 3050 60  0000 C CNN
+F 0 "SW1" H 6875 3050 60  0000 C CNN
 F 1 "SWITCH_SPST" V 6875 2580 60  0000 C CNN
 F 2 "molex_microclasp2:microclasp_vdrx2" H 6875 2900 60  0001 C CNN
@@
 	10350 1650 9600 1650
 $Comp
-L SWITCH_DPDT S?
+L SWITCH_DPDT S1
 U 1 1 5881AA8A
-P 5425 1300
-F 0 "S?" V 5305 950 60  0000 C CNN
-F 1 "SWITCH_DPDT" V 5305 1400 60  0000 C CNN
-F 2 "microclasp:microclasp_3" H 5425 1300 60  0001 C CNN
-F 3 "" H 5425 1300 60  0000 C CNN
-	1    5425 1300
+P 5350 1925
+F 0 "S1" V 5230 1575 60  0000 C CNN
+F 1 "SWITCH_DPDT" V 5230 2025 60  0000 C CNN
+F 2 "microclasp:microclasp_3" H 5350 1925 60  0001 C CNN
+F 3 "" H 5350 1925 60  0000 C CNN
+	1    5350 1925
 	0    1    1    0
 $EndComp
-Text Label 5105 1300 2    60   ~ 0
+Text Label 5030 1925 2    60   ~ 0
 V4
-Text Label 5745 1300 0    60   ~ 0
+Text Label 5670 1925 0    60   ~ 0
 GND
 Wire Wire Line
-	5125 1300 4925 1300
-Wire Wire Line
-	5725 1300 5945 1300
-Wire Wire Line
-	5425 1400 5425 1575
-Wire Wire Line
-	5425 1575 5950 1575
-Text Label 5475 1575 0    60   ~ 0
+	5050 1925 4850 1925
+Wire Wire Line
+	5650 1925 5870 1925
+Wire Wire Line
+	5350 2025 5350 2200
+Wire Wire Line
+	5350 2200 5875 2200
+Text Label 5400 2200 0    60   ~ 0
 Switch_on
 Text HLabel 1000 1125 0    60   Input ~ 0
@@
 Switch_on
 $Comp
-L RJ45 J?
+L RJ45 J1
 U 1 1 5881C2C5
 P 1925 4750
-F 0 "J?" H 2125 5250 50  0000 C CNN
+F 0 "J1" H 2125 5250 50  0000 C CNN
 F 1 "RJ45" H 1775 5250 50  0000 C CNN
-F 2 "" H 1925 4750 50  0000 C CNN
+F 2 "RJ45-SMD:TE-338088" H 1925 4750 50  0001 C CNN
 F 3 "" H 1925 4750 50  0000 C CNN
 	1    1925 4750
@@
 $EndComp
 $Comp
-L ZENERsmall D?
+L ZENERsmall D1
 U 1 1 58821700
 P 3220 1060
-F 0 "D?" H 3320 1020 50  0000 C CNN
+F 0 "D1" H 3320 1020 50  0000 C CNN
 F 1 "P6SMB30AT3G" H 3360 1180 50  0000 C CNN
 F 2 "Diodes_SMD:SMB_Standard" H 3220 1060 50  0001 C CNN
@@
 $EndComp
 $Comp
-L GND #PWR?
+L GND #PWR021
 U 1 1 58821707
 P 3220 1220
-F 0 "#PWR?" H 3220 970 50  0001 C CNN
+F 0 "#PWR021" H 3220 970 50  0001 C CNN
 F 1 "GND" H 3220 1070 50  0000 C CNN
 F 2 "" H 3220 1220 50  0000 C CNN
@@
 V24_in
 $Comp
-L Fuse F?
+L Fuse F1
 U 1 1 58821711
 P 2950 920
-F 0 "F?" V 3030 920 50  0000 C CNN
+F 0 "F1" V 3030 920 50  0000 C CNN
 F 1 "3413.0328.22" V 2875 920 50  0000 C CNN
 F 2 "dp_devices:dp_devices-C1206" V 2880 920 50  0001 C CNN

Commit message: Added a lot of things. Put a 5v to 4v buck as well as supporing the snapdragon board
Parts:
- removed J1: RJ45, RJ45-SMD:TE-338088, symbol RJ45
- added P13: CONN_02X15, symbol CONN_02X15
- SW1: footprint molex_microclasp2:microclasp_vdrx2 -> microclasp:microclasp_2
