File: connectors.sch (KiCad schematic (older format))
At the start: 11 parts, among them P1 Vbackup, P13 CONN_02X15, P2 CONN_02X05, P3 Hebi_1, P4 Hebi_2, SW1 SWITCH_SPST

Commit message: Cleaned up some wires and moved connectors out to main page. Also added some LEDs
Connections:
- net labels added: GND24
- wire segments 48 -> 49
Changed lines of the file:
@@
 LIBS:Sensors
 LIBS:LP3852-3.3
-LIBS:decaWave
+LIBS:0s102011ma1qn1
+LIBS:74LVC1G17
+LIBS:74V1T126
+LIBS:acs711klctr-12ab-t
+LIBS:AD7192
+LIBS:AD7193
+LIBS:am-hrr30-xxx
+LIBS:aon7528
+LIBS:AP7363
+LIBS:AS1359
+LIBS:csd16323q3
+LIBS:dmn2004dmk
+LIBS:dp_devices
+LIBS:DSPIC33E128MC506
+LIBS:fds6898az
+LIBS:ina197
+LIBS:irf7329pbf
+LIBS:ld1117
+LIBS:lm3478
+LIBS:lm3481
+LIBS:lt1910
+LIBS:ltc1871
+LIBS:ltc1982
+LIBS:MAG3110
+LIBS:mcp1700
+LIBS:mcp73831
+LIBS:mcsmt-g5030a1-3712
+LIBS:microchip_can
+LIBS:microclasp_hdrx2
+LIBS:microclasp_hdrx3
+LIBS:MPU-6000_MPU-6050
+LIBS:MPU-9150
+LIBS:nrf24l01+
+LIBS:pds1040l
+LIBS:pic12f1571
+LIBS:pinhead
+LIBS:psmn013-80ys
+LIBS:RESISTOR_ARRAY
+LIBS:rf803d
+LIBS:RGB_LED
+LIBS:Si1970DH
+LIBS:sn65hvd232
+LIBS:ssc54
+LIBS:sw_push_4
+LIBS:tc74
+LIBS:TPS2113A
+LIBS:tps54540
+LIBS:vs-mbrb1635pbf
+LIBS:xal5050-562meb
+LIBS:xal6030-182mec
 LIBS:conn_2x50
 LIBS:conn_open_q_x2
@@
 LIBS:ac-dc
 LIBS:actel
-LIBS:allegro
 LIBS:Altera
 LIBS:analog_devices
@@
 LIBS:logo
 LIBS:maxim
-LIBS:mechanical
 LIBS:microchip_dspic33dsc
 LIBS:microchip_pic10mcu
@@
 LIBS:microchip_pic32mcu
 LIBS:motor_drivers
-LIBS:motors
 LIBS:msp430
 LIBS:nordicsemi
@@
 LIBS:ttl_ieee
 LIBS:video
-LIBS:wiznet
 LIBS:Worldsemi
 LIBS:Xicor
-LIBS:zetex
 LIBS:Zilog
 LIBS:conn_2x45
@@
 Text Label 2020 2720 2    60   ~ 0
 V24_in
-$Comp
-L GNDPWR #PWR17
-U 1 1 5876C3D5
-P 1840 2170
-F 0 "#PWR17" H 1840 1970 50  0001 C CNN
-F 1 "GNDPWR" H 1840 2040 50  0000 C CNN
-F 2 "" H 1840 2120 50  0000 C CNN
-F 3 "" H 1840 2120 50  0000 C CNN
-	1    1840 2170
-	1    0    0    -1
-$EndComp
 Text Label 1640 2420 0    60   ~ 0
 signal_1s
@@
 Vbackup_in
 $Comp
-L GND #PWR18
+L GND #PWR018
 U 1 1 5876C3F8
 P 2130 3410
-F 0 "#PWR18" H 2130 3160 50  0001 C CNN
+F 0 "#PWR018" H 2130 3160 50  0001 C CNN
 F 1 "GND" H 2130 3260 50  0000 C CNN
 F 2 "" H 2130 3410 50  0000 C CNN
@@
 V_hebi1
 $Comp
-L GNDPWR #PWR16
+L GNDPWR #PWR019
 U 1 1 5876E2BA
 P 1835 4180
-F 0 "#PWR16" H 1835 3980 50  0001 C CNN
+F 0 "#PWR019" H 1835 3980 50  0001 C CNN
 F 1 "GNDPWR" H 1835 4050 50  0000 C CNN
 F 2 "" H 1835 4130 50  0000 C CNN
@@
 $EndComp
 $Comp
-L GNDPWR #PWR15
+L GNDPWR #PWR020
 U 1 1 5876E2C0
 P 1825 4620
-F 0 "#PWR15" H 1825 4420 50  0001 C CNN
+F 0 "#PWR020" H 1825 4420 50  0001 C CNN
 F 1 "GNDPWR" H 1825 4490 50  0000 C CNN
 F 2 "" H 1825 4570 50  0000 C CNN
@@
 Text Label 1345 5590 0    60   ~ 0
 Vmotors
-$Comp
-L GNDPWR #PWR19
-U 1 1 5876C3CF
-P 2680 2770
-F 0 "#PWR19" H 2680 2570 50  0001 C CNN
-F 1 "GNDPWR" H 2680 2640 50  0000 C CNN
-F 2 "" H 2680 2720 50  0000 C CNN
-F 3 "" H 2680 2720 50  0000 C CNN
-	1    2680 2770
-	1    0    0    -1
-$EndComp
 Text Label 10300 1440 2    60   ~ 0
 Vbackup_in
@@
 	2560 2720 2680 2720
 Wire Wire Line
-	2680 2720 2680 2770
-Wire Wire Line
 	2060 2720 1730 2720
 Wire Wire Line
@@
 Wire Wire Line
 	2020 2140 1840 2140
-Wire Wire Line
-	1840 2140 1840 2170
 Wire Wire Line
 	2560 2320 2890 2320
@@
 $EndComp
 $Comp
-L GND #PWR20
+L GND #PWR022
 U 1 1 58821707
 P 3220 1220
-F 0 "#PWR20" H 3220 970 50  0001 C CNN
+F 0 "#PWR022" H 3220 970 50  0001 C CNN
 F 1 "GND" H 3220 1070 50  0000 C CNN
 F 2 "" H 3220 1220 50  0000 C CNN
@@
 	1    0    0    -1
 $EndComp
+Text HLabel 1025 1250 0    60   Input ~ 0
+GND24
+Wire Wire Line
+	1025 1250 1350 1250
+Text Label 1075 1250 0    60   ~ 0
+GND24
+Wire Wire Line
+	2680 2720 2680 2770
+Wire Wire Line
+	1840 2140 1840 2170
+$Comp
+L GNDPWR #PWR017
+U 1 1 5876C3D5
+P 1840 2170
+F 0 "#PWR017" H 1840 1970 50  0001 C CNN
+F 1 "GNDPWR" H 1840 2040 50  0000 C CNN
+F 2 "" H 1840 2120 50  0000 C CNN
+F 3 "" H 1840 2120 50  0000 C CNN
+	1    1840 2170
+	1    0    0    -1
+$EndComp
+$Comp
+L GNDPWR #PWR021
+U 1 1 5876C3CF
+P 2680 2770
+F 0 "#PWR021" H 2680 2570 50  0001 C CNN
+F 1 "GNDPWR" H 2680 2640 50  0000 C CNN
+F 2 "" H 2680 2720 50  0000 C CNN
+F 3 "" H 2680 2720 50  0000 C CNN
+	1    2680 2770
+	1    0    0    -1
+$EndComp
