File: main_master_dev_boards/power_systems/power_on_switch/power_on_switch.sch (KiCad schematic (older format))
At the start: 14 parts, among them J1 Vbackup_in, J2 GND_in, J3 24_in, J4 Switch_out, J5 24_out, J6 GND_in, J7 GND_out, Q1 PSMN013-80YS, SW1 SW_Push, U1 LTC2955-1

Commit message: Modifying power switch dev board so that tracing and pads are bigger to make soldering easier.
Parts:
- J1, J3, J4, J5: footprint pinhead:pinhead-1X01 -> pinheaders:pinhead-01x01_3x1
- J2, J6, J7: footprint Pin_Headers:Pin_Header_Straight_1x01_Pitch2.54mm -> pinheaders:pinhead-01x01_3x1_square
Changed lines of the file:
@@
 LIBS:contrib
 LIBS:valves
-LIBS:antenna
-LIBS:AS1360
-LIBS:conn_2x45
-LIBS:conn_2x50
-LIBS:conn_open_q_x2
-LIBS:esd7c5
-LIBS:FDS4935A
-LIBS:FPF1203LUCX
-LIBS:lan9512
-LIBS:LMR16020
-LIBS:LP3852-3.3
-LIBS:LTC2955-1
-LIBS:MIC2026
-LIBS:Si1077X
-LIBS:Si1900DL
-LIBS:SN74LV1T125
-LIBS:SN74LV4T125
-LIBS:TDP6E001RSER
-LIBS:tps82084sil
-LIBS:TPS754
-LIBS:TPS61089
-LIBS:TPS61232DRC
-LIBS:TPS832130SIL
-LIBS:0s102011ma1qn1
-LIBS:74LVC1G17
-LIBS:74V1T126
-LIBS:acs711klctr-12ab-t
-LIBS:AD7192
-LIBS:AD7193
-LIBS:am-hrr30-xxx
-LIBS:aon7528
-LIBS:AP7363
-LIBS:AS1359
-LIBS:csd16323q3
-LIBS:dmn2004dmk
-LIBS:dp_devices
-LIBS:DSPIC33E128MC506
-LIBS:fds6898az
-LIBS:ina197
-LIBS:irf7329pbf
-LIBS:ld1117
-LIBS:lm3478
-LIBS:lm3481
-LIBS:lt1910
-LIBS:ltc1871
-LIBS:ltc1982
-LIBS:MAG3110
-LIBS:mcp1700
-LIBS:mcp73831
-LIBS:mcsmt-g5030a1-3712
-LIBS:microchip_can
-LIBS:microclasp_hdrx2
-LIBS:microclasp_hdrx3
-LIBS:MPU-6000_MPU-6050
-LIBS:MPU-9150
-LIBS:nrf24l01+
-LIBS:pds1040l
-LIBS:pic12f1571
-LIBS:pinhead
-LIBS:psmn013-80ys
-LIBS:RESISTOR_ARRAY
-LIBS:rf803d
-LIBS:RGB_LED
-LIBS:Si1970DH
-LIBS:sn65hvd232
-LIBS:ssc54
-LIBS:sw_push_4
-LIBS:tc74
-LIBS:tps54540
-LIBS:TPS2113A
-LIBS:vs-mbrb1635pbf
-LIBS:xal5050-562meb
-LIBS:xal6030-182mec
-LIBS:ld29150dt50r
-LIBS:ncp59151ds50r4g
-LIBS:pinhd-2x23
-LIBS:main_master_board-cache
-LIBS:main_master_board-rescue
+LIBS:power_on_switch-cache
 EELAYER 25 0
 EELAYER END
@@
 F 0 "J1" H 3170 2580 50  0000 C CNN
 F 1 "Vbackup_in" V 3270 2480 50  0000 C CNN
-F 2 "pinhead:pinhead-1X01" H 3170 2480 50  0001 C CNN
+F 2 "pinheaders:pinhead-01x01_3x1" H 3170 2480 50  0001 C CNN
 F 3 "" H 3170 2480 50  0001 C CNN
 	1    3170 2480
@@
 F 0 "J2" H 3460 2130 50  0000 C CNN
 F 1 "GND_in" V 3560 2030 50  0000 C CNN
-F 2 "Pin_Headers:Pin_Header_Straight_1x01_Pitch2.54mm" H 3460 2030 50  0001 C CNN
+F 2 "pinheaders:pinhead-01x01_3x1_square" H 3460 2030 50  0001 C CNN
 F 3 "" H 3460 2030 50  0001 C CNN
 	1    3460 2030
@@
 F 0 "J3" H 3710 3830 50  0000 C CNN
 F 1 "24_in" V 3810 3730 50  0000 C CNN
-F 2 "pinhead:pinhead-1X01" H 3710 3730 50  0001 C CNN
+F 2 "pinheaders:pinhead-01x01_3x1" H 3710 3730 50  0001 C CNN
 F 3 "" H 3710 3730 50  0001 C CNN
 	1    3710 3730
@@
 F 0 "J5" H 6115 3880 50  0000 C CNN
 F 1 "24_out" V 6215 3780 50  0000 C CNN
-F 2 "pinhead:pinhead-1X01" H 6115 3780 50  0001 C CNN
+F 2 "pinheaders:pinhead-01x01_3x1" H 6115 3780 50  0001 C CNN
 F 3 "" H 6115 3780 50  0001 C CNN
 	1    6115 3780
@@
 F 0 "J4" H 6065 3580 50  0000 C CNN
 F 1 "Switch_out" V 6165 3480 50  0000 C CNN
-F 2 "pinhead:pinhead-1X01" H 6065 3480 50  0001 C CNN
+F 2 "pinheaders:pinhead-01x01_3x1" H 6065 3480 50  0001 C CNN
 F 3 "" H 6065 3480 50  0001 C CNN
 	1    6065 3480
@@
 F 0 "J7" H 6105 4240 50  0000 C CNN
 F 1 "GND_out" V 6205 4140 50  0000 C CNN
-F 2 "Pin_Headers:Pin_Header_Straight_1x01_Pitch2.54mm" H 6105 4140 50  0001 C CNN
+F 2 "pinheaders:pinhead-01x01_3x1_square" H 6105 4140 50  0001 C CNN
 F 3 "" H 6105 4140 50  0001 C CNN
 	1    6105 4140
@@
 F 0 "J6" H 3695 4240 50  0000 C CNN
 F 1 "GND_in" V 3795 4140 50  0000 C CNN
-F 2 "Pin_Headers:Pin_Header_Straight_1x01_Pitch2.54mm" H 3695 4140 50  0001 C CNN
+F 2 "pinheaders:pinhead-01x01_3x1_square" H 3695 4140 50  0001 C CNN
 F 3 "" H 3695 4140 50  0001 C CNN
 	1    3695 4140
