File: main_master_dev_boards/power_systems/power_4_to_5/power_4_to_5.sch (KiCad schematic (older format))
At the start: 18 parts

Commit message: Added and updated 4_to_5 dev boards files
Parts:
- removed C?: 4.7uF, Capacitors_SMD:C_0603, symbol C_Small
- removed C?: 47uF, Capacitors_SMD:C_1206, symbol C
- removed R?: 10K, Resistors_SMD:R_0603, symbol R_Small
- removed R?: 10K, Resistors_SMD:R_0603, symbol R
- added C6, C7, C8: 22uF, Capacitors_SMD:C_0805_HandSoldering, symbol C
- added P1: Vbackup, pinheaders:pinhead-01x01_3x1, symbol CONN_01X01
- added P2, P5: GND, pinheaders:pinhead-01x01_3x1_square, symbol CONN_01X01
- added P3: 5V_Main, pinheaders:pinhead-01x01_3x1, symbol CONN_01X01
- added P4: PG_5V_Main, pinheaders:pinhead-01x01_3x1, symbol CONN_01X01
- added P6: V5_Backup, pinheaders:pinhead-01x01_3x1, symbol CONN_01X01
- added R4: 402K, Resistors_SMD:R_0805_HandSoldering, symbol R_Small
- added R5: 100K, Resistors_SMD:R_0805_HandSoldering, symbol R_Small
- added U2: Si1900DL, NASA_IRG_SSB:SOT323-6, symbol Si1900DL
- added U3: SN74LVC1G04, TO_SOT_Packages_SMD:SOT-23-5_HandSoldering, symbol SN74LVC1G04
- C1, C2, C3: renamed from C?; footprint Capacitors_SMD:C_0603 -> Capacitors_SMD:C_0805_HandSoldering
- C4: renamed from C?; footprint Capacitors_SMD:C_0805 -> Capacitors_SMD:C_0805_HandSoldering; Field5 JMK212BJ226MG-T -> (none); Voltage 6.3V -> (none)
- C5: renamed from C?; value 15nF -> 10nF; footprint Capacitors_SMD:C_0402 -> Capacitors_SMD:C_0805_HandSoldering; Field5 GRM155R71C153KA01D -> (none); Voltage 16V -> (none)
- D1, D2: renamed from D?; footprint (none) -> LEDs:LED_0805
- L1: renamed from L?; footprint IHLP-2020BZ:IHLP-2020BZ -> XFL4020:XFL4020; Field5 IHLP2020BZER1R0M11 -> XFL4020-102MEB; Resistance 0.018 Ohms -> (none)
- R1, R6: renamed from R?; footprint (none) -> Resistors_SMD:R_0805_HandSoldering
- R2: renamed from R?; value 200 -> 470; footprint Resistors_SMD:R_0603 -> Resistors_SMD:R_0805_HandSoldering
- R3: renamed from R?; footprint Resistors_SMD:R_0603 -> Resistors_SMD:R_0805_HandSoldering
- gave numbers to parts that had none: 2
Connections:
- net labels added: PG_5V_MAIN, PROG, V5_Main, ~PG_5V_MAIN
- net labels removed: Switch_on, V5, Vss, charge_on, charging
- wire segments 72 -> 65
- no-connect marks 1 -> 2
Other:
- note added: "PROG:\n2K to GND = ON\nFLOAT = OFF"
- note removed: "Vbackup Buck EN\nLiPo Charger ~EN\n"
- moved on the sheet: C1, C2, C3, D1, IC1, R1, R2
