File: main_board/main_board_onion/batteryMonitor.sch (KiCad schematic (older format))
At the start: 46 parts, among them J12 Battery Input Connector, Q2 PSMN5R8-40YS, Q3 IRLML6402, Q4 PSMN5R8-40YS, Q5 PSMN5R8-40YS, U5 BQ76930

Commit message: Finished initial routing of this design
Parts:
- C10, C11, C12, C13, C14, C15, C16, C17, C18, C19, C20, C21, C24, C8, C9: footprint Capacitor_SMD:C_0603_1608Metric -> Capacitor_SMD:C_0402_1005Metric
- R14, R15, R16, R17, R18, R19, R20, R21, R22, R24, R26, R27, R28, R30, R31: footprint Resistor_SMD:R_0603_1608Metric -> Resistor_SMD:R_0402_1005Metric
Changed lines of the file:
@@
 $Descr A4 11693 8268
 encoding utf-8
-Sheet 3 7
+Sheet 7 7
 Title ""
 Date ""
@@
 F 0 "R14" V 1525 2350 50  0000 C CNN
 F 1 "1k" V 1625 2350 50  0000 C CNN
-F 2 "Resistor_SMD:R_0603_1608Metric" V 1555 2350 50  0001 C CNN
+F 2 "Resistor_SMD:R_0402_1005Metric" V 1555 2350 50  0001 C CNN
 F 3 "~" H 1625 2350 50  0001 C CNN
 	1    1625 2350
@@
 F 0 "C8" H 1992 2496 50  0000 L CNN
 F 1 "1uF" H 1992 2405 50  0000 L CNN
-F 2 "Capacitor_SMD:C_0603_1608Metric" H 1900 2450 50  0001 C CNN
+F 2 "Capacitor_SMD:C_0402_1005Metric" H 1900 2450 50  0001 C CNN
 F 3 "~" H 1900 2450 50  0001 C CNN
 	1    1900 2450
@@
 F 0 "R26" V 5400 2725 50  0000 C CNN
 F 1 "10k" V 5475 2725 50  0000 C CNN
-F 2 "Resistor_SMD:R_0603_1608Metric" V 5405 2725 50  0001 C CNN
+F 2 "Resistor_SMD:R_0402_1005Metric" V 5405 2725 50  0001 C CNN
 F 3 "~" H 5475 2725 50  0001 C CNN
 	1    5475 2725
@@
 F 0 "R27" V 5700 3575 50  0000 C CNN
 F 1 "10k" V 5775 3575 50  0000 C CNN
-F 2 "Resistor_SMD:R_0603_1608Metric" V 5705 3575 50  0001 C CNN
+F 2 "Resistor_SMD:R_0402_1005Metric" V 5705 3575 50  0001 C CNN
 F 3 "~" H 5775 3575 50  0001 C CNN
 	1    5775 3575
@@
 F 0 "C21" V 5650 3625 50  0000 C CNN
 F 1 "1uF" V 5575 3625 50  0000 C CNN
-F 2 "Capacitor_SMD:C_0603_1608Metric" H 5475 3625 50  0001 C CNN
+F 2 "Capacitor_SMD:C_0402_1005Metric" H 5475 3625 50  0001 C CNN
 F 3 "~" H 5475 3625 50  0001 C CNN
 	1    5475 3625
@@
 Wire Wire Line
 	5575 3625 5650 3625
-$Comp
-L Device:C_Small C20
-U 1 1 5CBEB518
-P 5475 3025
-F 0 "C20" V 5650 3025 50  0000 C CNN
-F 1 "1uF" V 5575 3025 50  0000 C CNN
-F 2 "Capacitor_SMD:C_0603_1608Metric" H 5475 3025 50  0001 C CNN
-F 3 "~" H 5475 3025 50  0001 C CNN
-	1    5475 3025
-	0    1    1    0
-$EndComp
 Wire Wire Line
 	5150 3025 5375 3025
@@
 F 0 "R31" V 6775 2825 50  0000 C CNN
 F 1 "100" V 6850 2825 50  0000 C CNN
-F 2 "Resistor_SMD:R_0603_1608Metric" V 6780 2825 50  0001 C CNN
+F 2 "Resistor_SMD:R_0402_1005Metric" V 6780 2825 50  0001 C CNN
 F 3 "~" H 6850 2825 50  0001 C CNN
 	1    6850 2825
@@
 F 0 "R30" V 6550 2250 50  0000 C CNN
 F 1 "100" V 6625 2250 50  0000 C CNN
-F 2 "Resistor_SMD:R_0603_1608Metric" V 6555 2250 50  0001 C CNN
+F 2 "Resistor_SMD:R_0402_1005Metric" V 6555 2250 50  0001 C CNN
 F 3 "~" H 6625 2250 50  0001 C CNN
 	1    6625 2250
@@
 F 0 "C24" H 7175 2850 50  0000 L CNN
 F 1 "1uF" H 7150 2750 50  0000 L CNN
-F 2 "Capacitor_SMD:C_0603_1608Metric" H 7375 2800 50  0001 C CNN
+F 2 "Capacitor_SMD:C_0402_1005Metric" H 7375 2800 50  0001 C CNN
 F 3 "~" H 7375 2800 50  0001 C CNN
 	1    7375 2800
@@
 F 0 "C17" V 2875 4825 50  0000 L CNN
 F 1 "0.1Uf" V 2650 4775 50  0000 L CNN
-F 2 "Capacitor_SMD:C_0603_1608Metric" H 2775 4875 50  0001 C CNN
+F 2 "Capacitor_SMD:C_0402_1005Metric" H 2775 4875 50  0001 C CNN
 F 3 "~" H 2775 4875 50  0001 C CNN
 	1    2775 4875
@@
 F 0 "C18" V 3125 4825 50  0000 L CNN
 F 1 "0.1Uf" V 2900 4775 50  0000 L CNN
-F 2 "Capacitor_SMD:C_0603_1608Metric" H 3025 4875 50  0001 C CNN
+F 2 "Capacitor_SMD:C_0402_1005Metric" H 3025 4875 50  0001 C CNN
 F 3 "~" H 3025 4875 50  0001 C CNN
 	1    3025 4875
@@
 F 0 "C16" V 2625 4825 50  0000 L CNN
 F 1 "0.1Uf" V 2400 4775 50  0000 L CNN
-F 2 "Capacitor_SMD:C_0603_1608Metric" H 2525 4875 50  0001 C CNN
+F 2 "Capacitor_SMD:C_0402_1005Metric" H 2525 4875 50  0001 C CNN
 F 3 "~" H 2525 4875 50  0001 C CNN
 	1    2525 4875
@@
 F 0 "R22" H 2600 5225 50  0000 L CNN
 F 1 "100" V 2550 5150 50  0000 L CNN
-F 2 "Resistor_SMD:R_0603_1608Metric" V 2480 5225 50  0001 C CNN
+F 2 "Resistor_SMD:R_0402_1005Metric" V 2480 5225 50  0001 C CNN
 F 3 "~" H 2550 5225 50  0001 C CNN
 	1    2550 5225
@@
 F 0 "R24" H 3050 5225 50  0000 L CNN
 F 1 "100" V 3000 5150 50  0000 L CNN
-F 2 "Resistor_SMD:R_0603_1608Metric" V 2930 5225 50  0001 C CNN
+F 2 "Resistor_SMD:R_0402_1005Metric" V 2930 5225 50  0001 C CNN
 F 3 "~" H 3000 5225 50  0001 C CNN
 	1    3000 5225
@@
 F 0 "R15" V 1525 2550 50  0000 C CNN
 F 1 "1k" V 1625 2550 50  0000 C CNN
-F 2 "Resistor_SMD:R_0603_1608Metric" V 1555 2550 50  0001 C CNN
+F 2 "Resistor_SMD:R_0402_1005Metric" V 1555 2550 50  0001 C CNN
 F 3 "~" H 1625 2550 50  0001 C CNN
 	1    1625 2550
@@
 F 0 "R16" V 1525 2750 50  0000 C CNN
 F 1 "1k" V 1625 2750 50  0000 C CNN
-F 2 "Resistor_SMD:R_0603_1608Metric" V 1555 2750 50  0001 C CNN
+F 2 "Resistor_SMD:R_0402_1005Metric" V 1555 2750 50  0001 C CNN
 F 3 "~" H 1625 2750 50  0001 C CNN
 	1    1625 2750
@@
 F 0 "R17" V 1525 3150 50  0000 C CNN
 F 1 "1k" V 1625 3150 50  0000 C CNN
-F 2 "Resistor_SMD:R_0603_1608Metric" V 1555 3150 50  0001 C CNN
+F 2 "Resistor_SMD:R_0402_1005Metric" V 1555 3150 50  0001 C CNN
 F 3 "~" H 1625 3150 50  0001 C CNN
 	1    1625 3150
@@
 F 0 "R18" V 1525 3350 50  0000 C CNN
 F 1 "1k" V 1625 3350 50  0000 C CNN
-F 2 "Resistor_SMD:R_0603_1608Metric" V 1555 3350 50  0001 C CNN
+F 2 "Resistor_SMD:R_0402_1005Metric" V 1555 3350 50  0001 C CNN
 F 3 "~" H 1625 3350 50  0001 C CNN
 	1    1625 3350
@@
 F 0 "R19" V 1525 3550 50  0000 C CNN
 F 1 "1k" V 1625 3550 50  0000 C CNN
-F 2 "Resistor_SMD:R_0603_1608Metric" V 1555 3550 50  0001 C CNN
+F 2 "Resistor_SMD:R_0402_1005Metric" V 1555 3550 50  0001 C CNN
 F 3 "~" H 1625 3550 50  0001 C CNN
 	1    1625 3550
@@
 F 0 "R20" V 1525 3750 50  0000 C CNN
 F 1 "1k" V 1625 3750 50  0000 C CNN
-F 2 "Resistor_SMD:R_0603_1608Metric" V 1555 3750 50  0001 C CNN
+F 2 "Resistor_SMD:R_0402_1005Metric" V 1555 3750 50  0001 C CNN
 F 3 "~" H 1625 3750 50  0001 C CNN
 	1    1625 3750
@@
 F 0 "C9" H 1992 2696 50  0000 L CNN
 F 1 "1uF" H 1992 2605 50  0000 L CNN
-F 2 "Capacitor_SMD:C_0603_1608Metric" H 1900 2650 50  0001 C CNN
+F 2 "Capacitor_SMD:C_0402_1005Metric" H 1900 2650 50  0001 C CNN
 F 3 "~" H 1900 2650 50  0001 C CNN
 	1    1900 2650
@@
 F 0 "C10" H 1992 2896 50  0000 L CNN
 F 1 "1uF" H 1992 2805 50  0000 L CNN
-F 2 "Capacitor_SMD:C_0603_1608Metric" H 1900 2850 50  0001 C CNN
+F 2 "Capacitor_SMD:C_0402_1005Metric" H 1900 2850 50  0001 C CNN
 F 3 "~" H 1900 2850 50  0001 C CNN
 	1    1900 2850
@@
 F 0 "C11" H 1992 3096 50  0000 L CNN
 F 1 "1uF" H 1992 3005 50  0000 L CNN
-F 2 "Capacitor_SMD:C_0603_1608Metric" H 1900 3050 50  0001 C CNN
+F 2 "Capacitor_SMD:C_0402_1005Metric" H 1900 3050 50  0001 C CNN
 F 3 "~" H 1900 3050 50  0001 C CNN
 	1    1900 3050
@@
 F 0 "C12" H 1992 3496 50  0000 L CNN
 F 1 "1uF" H 1992 3405 50  0000 L CNN
-F 2 "Capacitor_SMD:C_0603_1608Metric" H 1900 3450 50  0001 C CNN
+F 2 "Capacitor_SMD:C_0402_1005Metric" H 1900 3450 50  0001 C CNN
 F 3 "~" H 1900 3450 50  0001 C CNN
 	1    1900 3450
@@
 F 0 "C13" H 1992 3696 50  0000 L CNN
 F 1 "1uF" H 1992 3605 50  0000 L CNN
-F 2 "Capacitor_SMD:C_0603_1608Metric" H 1900 3650 50  0001 C CNN
+F 2 "Capacitor_SMD:C_0402_1005Metric" H 1900 3650 50  0001 C CNN
 F 3 "~" H 1900 3650 50  0001 C CNN
 	1    1900 3650
@@
 F 0 "C14" H 1992 3896 50  0000 L CNN
 F 1 "1uF" H 1992 3805 50  0000 L CNN
-F 2 "Capacitor_SMD:C_0603_1608Metric" H 1900 3850 50  0001 C CNN
+F 2 "Capacitor_SMD:C_0402_1005Metric" H 1900 3850 50  0001 C CNN
 F 3 "~" H 1900 3850 50  0001 C CNN
 	1    1900 3850
@@
 F 0 "C15" H 1992 4096 50  0000 L CNN
 F 1 "1uF" H 1992 4005 50  0000 L CNN
-F 2 "Capacitor_SMD:C_0603_1608Metric" H 1900 4050 50  0001 C CNN
+F 2 "Capacitor_SMD:C_0402_1005Metric" H 1900 4050 50  0001 C CNN
 F 3 "~" H 1900 4050 50  0001 C CNN
 	1    1900 4050
@@
 F 0 "R21" V 1525 4150 50  0000 C CNN
 F 1 "1k" V 1625 4150 50  0000 C CNN
-F 2 "Resistor_SMD:R_0603_1608Metric" V 1555 4150 50  0001 C CNN
+F 2 "Resistor_SMD:R_0402_1005Metric" V 1555 4150 50  0001 C CNN
 F 3 "~" H 1625 4150 50  0001 C CNN
 	1    1625 4150
@@
 F 0 "C19" H 3367 1896 50  0000 L CNN
 F 1 "4.7uF" H 3367 1805 50  0000 L CNN
-F 2 "Capacitor_SMD:C_0603_1608Metric" H 3275 1850 50  0001 C CNN
+F 2 "Capacitor_SMD:C_0402_1005Metric" H 3275 1850 50  0001 C CNN
 F 3 "~" H 3275 1850 50  0001 C CNN
 	1    3275 1850
@@
 F 0 "R28" V 5925 3425 50  0000 C CNN
 F 1 "10k" V 6000 3425 50  0000 C CNN
-F 2 "Resistor_SMD:R_0603_1608Metric" V 5930 3425 50  0001 C CNN
+F 2 "Resistor_SMD:R_0402_1005Metric" V 5930 3425 50  0001 C CNN
 F 3 "~" H 6000 3425 50  0001 C CNN
 	1    6000 3425
@@
 Text HLabel 6800 3525 2    50   Input ~ 0
 Button_R
+$Comp
+L Device:C_Small C20
+U 1 1 5CBEB518
+P 5475 3025
+F 0 "C20" V 5650 3025 50  0000 C CNN
+F 1 "1uF" V 5575 3025 50  0000 C CNN
+F 2 "Capacitor_SMD:C_0402_1005Metric" H 5475 3025 50  0001 C CNN
+F 3 "~" H 5475 3025 50  0001 C CNN
+	1    5475 3025
+	0    1    1    0
+$EndComp
 $EndSCHEMATC

Commit message: Added Gerber files for the version uploaded to MacroFab for manufacturing. Plus small changes made before uploading it.
Parts:
- C10, C11, C12, C13, C14, C15, C20, C21, C24, C8, C9: Field4 (none) -> MF-CAP-0402-1uF
Changed lines of the file:
@@
 F 2 "Capacitor_SMD:C_0402_1005Metric" H 1900 2450 50  0001 C CNN
 F 3 "~" H 1900 2450 50  0001 C CNN
+F 4 "" H 1900 2450 50  0001 C CNN "Mouser Part Number"
+F 5 "" H 1900 2450 50  0001 C CNN "Description"
+F 6 "MF-CAP-0402-1uF" H 1900 2450 50  0001 C CNN "Field4"
 	1    1900 2450
 	1    0    0    -1
@@
 F 2 "Capacitor_SMD:C_0402_1005Metric" H 5475 3625 50  0001 C CNN
 F 3 "~" H 5475 3625 50  0001 C CNN
+F 4 "" H 5475 3625 50  0001 C CNN "Mouser Part Number"
+F 5 "" H 5475 3625 50  0001 C CNN "Description"
+F 6 "MF-CAP-0402-1uF" H 5475 3625 50  0001 C CNN "Field4"
 	1    5475 3625
 	0    1    1    0
@@
 F 2 "Capacitor_SMD:C_0402_1005Metric" H 7375 2800 50  0001 C CNN
 F 3 "~" H 7375 2800 50  0001 C CNN
+F 4 "" H 7375 2800 50  0001 C CNN "Mouser Part Number"
+F 5 "" H 7375 2800 50  0001 C CNN "Description"
+F 6 "MF-CAP-0402-1uF" H 7375 2800 50  0001 C CNN "Field4"
 	1    7375 2800
 	-1   0    0    1
@@
 F 2 "Capacitor_SMD:C_0402_1005Metric" H 1900 2650 50  0001 C CNN
 F 3 "~" H 1900 2650 50  0001 C CNN
+F 4 "" H 1900 2650 50  0001 C CNN "Mouser Part Number"
+F 5 "" H 1900 2650 50  0001 C CNN "Description"
+F 6 "MF-CAP-0402-1uF" H 1900 2650 50  0001 C CNN "Field4"
 	1    1900 2650
 	1    0    0    -1
@@
 F 2 "Capacitor_SMD:C_0402_1005Metric" H 1900 2850 50  0001 C CNN
 F 3 "~" H 1900 2850 50  0001 C CNN
+F 4 "" H 1900 2850 50  0001 C CNN "Mouser Part Number"
+F 5 "" H 1900 2850 50  0001 C CNN "Description"
+F 6 "MF-CAP-0402-1uF" H 1900 2850 50  0001 C CNN "Field4"
 	1    1900 2850
 	1    0    0    -1
@@
 F 2 "Capacitor_SMD:C_0402_1005Metric" H 1900 3050 50  0001 C CNN
 F 3 "~" H 1900 3050 50  0001 C CNN
+F 4 "" H 1900 3050 50  0001 C CNN "Mouser Part Number"
+F 5 "" H 1900 3050 50  0001 C CNN "Description"
+F 6 "MF-CAP-0402-1uF" H 1900 3050 50  0001 C CNN "Field4"
 	1    1900 3050
 	1    0    0    -1
@@
 F 2 "Capacitor_SMD:C_0402_1005Metric" H 1900 3450 50  0001 C CNN
 F 3 "~" H 1900 3450 50  0001 C CNN
+F 4 "" H 1900 3450 50  0001 C CNN "Mouser Part Number"
+F 5 "" H 1900 3450 50  0001 C CNN "Description"
+F 6 "MF-CAP-0402-1uF" H 1900 3450 50  0001 C CNN "Field4"
 	1    1900 3450
 	1    0    0    -1
@@
 F 2 "Capacitor_SMD:C_0402_1005Metric" H 1900 3650 50  0001 C CNN
 F 3 "~" H 1900 3650 50  0001 C CNN
+F 4 "" H 1900 3650 50  0001 C CNN "Mouser Part Number"
+F 5 "" H 1900 3650 50  0001 C CNN "Description"
+F 6 "MF-CAP-0402-1uF" H 1900 3650 50  0001 C CNN "Field4"
 	1    1900 3650
 	1    0    0    -1
@@
 F 2 "Capacitor_SMD:C_0402_1005Metric" H 1900 3850 50  0001 C CNN
 F 3 "~" H 1900 3850 50  0001 C CNN
+F 4 "" H 1900 3850 50  0001 C CNN "Mouser Part Number"
+F 5 "" H 1900 3850 50  0001 C CNN "Description"
+F 6 "MF-CAP-0402-1uF" H 1900 3850 50  0001 C CNN "Field4"
 	1    1900 3850
 	1    0    0    -1
@@
 F 2 "Capacitor_SMD:C_0402_1005Metric" H 1900 4050 50  0001 C CNN
 F 3 "~" H 1900 4050 50  0001 C CNN
+F 4 "" H 1900 4050 50  0001 C CNN "Mouser Part Number"
+F 5 "" H 1900 4050 50  0001 C CNN "Description"
+F 6 "MF-CAP-0402-1uF" H 1900 4050 50  0001 C CNN "Field4"
 	1    1900 4050
 	1    0    0    -1
@@
 F 2 "Capacitor_SMD:C_0402_1005Metric" H 5475 3025 50  0001 C CNN
 F 3 "~" H 5475 3025 50  0001 C CNN
+F 4 "" H 5475 3025 50  0001 C CNN "Mouser Part Number"
+F 5 "" H 5475 3025 50  0001 C CNN "Description"
+F 6 "MF-CAP-0402-1uF" H 5475 3025 50  0001 C CNN "Field4"
 	1    5475 3025
 	0    1    1    0

Commit message: went back to original Macrofab v2 files and made changes for v3.5
Parts:
- removed R28: 10k, Resistor_SMD:R_0402_1005Metric, symbol Device:R
Connections:
- wire segments 183 -> 188
Other:
- moved on the sheet: R21
Changed lines of the file:
@@
-EESchema Schematic File Version 5
+EESchema Schematic File Version 4
 LIBS:main_board_onion-cache
-EELAYER 29 0
+EELAYER 30 0
 EELAYER END
 $Descr A4 11693 8268
@@
 	1    0    0    -1
 $EndComp
-Text Label 1775 3950 2    50   ~ 0
+Text Label 1450 3950 2    50   ~ 0
 Batt_GND
 Wire Wire Line
-	1475 4150 1425 4150
-Wire Wire Line
 	1475 3750 1300 3750
-Wire Wire Line
-	1900 3950 1425 3950
 Wire Wire Line
 	1475 3550 1300 3550
@@
 	2300 3925 3475 3925
 Wire Wire Line
-	2325 4150 2325 4075
-Wire Wire Line
-	2325 4075 3475 4075
-Wire Wire Line
 	1475 3150 1425 3150
 Wire Wire Line
@@
 Wire Wire Line
 	2325 3350 2325 3325
-Wire Wire Line
-	2325 3325 3475 3325
 Text Label 2325 3325 0    50   ~ 0
 VC5
@@
 	2650 4225 2650 4875
 Wire Wire Line
-	1425 4150 1425 5400
-Wire Wire Line
 	1425 5400 2250 5400
-Connection ~ 1425 4150
-Wire Wire Line
-	1425 4150 1050 4150
 Connection ~ 2550 5400
 Wire Wire Line
@@
 	1    0    0    -1
 $EndComp
-Connection ~ 1900 3950
-Wire Wire Line
-	1900 4150 2325 4150
-$Comp
-L Device:R R21
-U 1 1 5CBA554C
-P 1625 4150
-F 0 "R21" V 1525 4150 50  0000 C CNN
-F 1 "1k" V 1625 4150 50  0000 C CNN
-F 2 "Resistor_SMD:R_0402_1005Metric" V 1555 4150 50  0001 C CNN
-F 3 "~" H 1625 4150 50  0001 C CNN
-	1    1625 4150
-	0    1    1    0
-$EndComp
-Wire Wire Line
-	1775 4150 1900 4150
-Connection ~ 1900 4150
 $Comp
 L Transistor_FET:IRLML6402 Q3
@@
 	5650 3725 5775 3725
 Connection ~ 5775 3725
-$Comp
-L Device:R R28
-U 1 1 5CBD875C
-P 6000 3425
-F 0 "R28" V 5925 3425 50  0000 C CNN
-F 1 "10k" V 6000 3425 50  0000 C CNN
-F 2 "Resistor_SMD:R_0402_1005Metric" V 5930 3425 50  0001 C CNN
-F 3 "~" H 6000 3425 50  0001 C CNN
-	1    6000 3425
-	0    1    1    0
-$EndComp
-Wire Wire Line
-	5850 3425 5775 3425
 Connection ~ 5775 3425
 Wire Wire Line
@@
 Text Label 2375 3925 0    50   ~ 0
 VC1
-Text Label 6750 3525 2    50   ~ 0
+Text Label 6450 3525 2    50   ~ 0
 VC1
 Wire Wire Line
-	6800 3525 6600 3525
+	6500 3525 6300 3525
 Text Notes 3125 6900 0    50   ~ 0
 cell minimum volatage	3.0V\ncell count	6\ncharge voltage	25.2\nmax charge current	1.75A\npeak discharge current	20A\nOV Proteciton threshold	4.3V\nOV protection Delay	2s\nUV Protection Threshold	2.5V\nUV protection Delay	2s\nOCD Protection Threshold 	20A -> PROTECT2[0:3] = 0xD (89mV, 19.3A, RSNS = 1)\nOCD Protection Delay	320ms -> PROTECT2[4:6] = 0x5 (320ms)\nSCD Protection Threshold	35A -> PROTECT1[0:2] = 0x5 (155mV, 33.6A, RSNS = 1)\nSCD Protection Delay	100us -> PROTECT1[3:4] = 0X1 (100us)
 Wire Wire Line
-	2325 3775 3475 3775
+	2325 3775 3125 3775
 $Comp
 L battery_management:BQ76930 U5
@@
 $EndComp
 Wire Wire Line
-	2325 2875 3475 2875
-Text Label 3425 3625 2    50   ~ 0
-low_GND
-Text Label 3425 3475 2    50   ~ 0
-low_GND
+	2325 2875 3100 2875
 Wire Wire Line
 	3475 3475 3125 3475
 Wire Wire Line
 	3475 3625 3125 3625
-Text Label 3425 2725 2    50   ~ 0
-low_GND
-Text Label 3425 2575 2    50   ~ 0
-low_GND
 Wire Wire Line
 	3475 2575 3100 2575
@@
 Text HLabel 10050 2425 2    50   Output ~ 0
 PACK_GND
-Wire Wire Line
-	6150 3425 6800 3425
-Text HLabel 6800 3425 2    50   Input ~ 0
+Text HLabel 6500 3425 2    50   Input ~ 0
 Button_L
-Text HLabel 6800 3525 2    50   Input ~ 0
+Text HLabel 6500 3525 2    50   Input ~ 0
 Button_R
 $Comp
@@
 	0    1    1    0
 $EndComp
+Wire Wire Line
+	3100 2575 3100 2725
+Wire Wire Line
+	3100 2725 3100 2875
+Connection ~ 3100 2725
+Connection ~ 3100 2875
+Wire Wire Line
+	3100 2875 3475 2875
+$Comp
+L Device:R R21
+U 1 1 5CBA554C
+P 1625 3950
+F 0 "R21" V 1525 3950 50  0000 C CNN
+F 1 "1k" V 1625 3950 50  0000 C CNN
+F 2 "Resistor_SMD:R_0402_1005Metric" V 1555 3950 50  0001 C CNN
+F 3 "~" H 1625 3950 50  0001 C CNN
+	1    1625 3950
+	0    1    1    0
+$EndComp
+Wire Wire Line
+	1425 4150 1050 4150
+Connection ~ 1425 4150
+Wire Wire Line
+	1425 4150 1425 5400
+Wire Wire Line
+	1425 4150 1900 4150
+Wire Wire Line
+	1775 3950 1900 3950
+Connection ~ 1900 3950
+Wire Wire Line
+	1475 3950 1100 3950
+Wire Wire Line
+	1900 3950 2300 3950
+Wire Wire Line
+	2300 3950 2300 4075
+Wire Wire Line
+	2300 4075 3475 4075
+Wire Wire Line
+	2325 3325 3475 3325
+Wire Wire Line
+	3125 3475 3125 3625
+Wire Wire Line
+	3125 3625 3125 3775
+Connection ~ 3125 3625
+Connection ~ 3125 3775
+Wire Wire Line
+	3125 3775 3475 3775
+Wire Wire Line
+	5775 3425 6500 3425
 $EndSCHEMATC
